File: CAD/MaxSensorComplete.sch (KiCad schematic (older format))
At the start: 17 parts

Commit message: Finished PCB Draft -- waiting for review
Parts:
- removed C1, C2: 1µF, symbol Device:C
- removed R1, R2, R3, R4, R5: 4.7k, symbol Device:R
- removed U?: MAX30102EFD+, symbol Sensor2:MAX30102EFD+
- removed U?: MAX14595ETA+, symbol Sensor2:MAX14595ETA+
- added C15: 10µF 10V, Capacitor_SMD:C_0402_1005Metric, symbol Device:C
- added C17, C27: 22u, Capacitor_SMD:C_0603_1608Metric, symbol Device:C
- added C26: 1µf 10V, Capacitor_SMD:C_0402_1005Metric, symbol Device:C
- added D5: LED-LT PWSG-AABB-36-46-F, LED_SMD:LED_PLCC-2, symbol Device:LED
- added D6, D8: VEMD5010X01, footprints:VEMD5010X01, symbol VEMD5010X01:VEMD5010X01
- added D7: LED_LY_P47F-TM, LED_SMD:LED_PLCC-2, symbol Device:LED
- added R26, R27, R28, R29, R30: 50k, Resistor_SMD:R_0402_1005Metric, symbol Device:R
- added R36: 0, Resistor_SMD:R_0603_1608Metric, symbol Device:R
- added U7: TXB0104RUT, Package_DFN_QFN:Texas_R_PUQFN-N12, symbol Logic_LevelTranslator:TXB0104RUT
- added U9: MAX86141ENP+, footprints:MAX86141ENP, symbol MAX86141ENP:MAX86141ENP+
- C11: renamed from C6; footprint (none) -> Capacitor_SMD:C_0402_1005Metric
- C12: renamed from C3; footprint (none) -> Capacitor_SMD:C_0402_1005Metric
- C13: renamed from C7; footprint (none) -> Capacitor_SMD:C_0402_1005Metric
- C14: renamed from C5; footprint (none) -> Capacitor_SMD:C_0402_1005Metric
- C16: renamed from C4; footprint (none) -> Capacitor_SMD:C_0402_1005Metric
- L2: renamed from L1; footprint (none) -> Inductor_SMD:L_0603_1608Metric
- R31: renamed from R6; footprint (none) -> Resistor_SMD:R_0402_1005Metric
- U8: renamed from U?; footprint (none) -> footprints:MAX1921EUT18&plus_T
Connections:
- net labels added: +3V3, CSB, CSB_O, SCLK, SCLK_O, SDI, SDI_O, SDO, SDO_O, VCC
- net labels removed: INT, SCL, SDA, Vin
- wire segments 88 -> 122
Other:
- note added: "Ground line should be routerd separately to the connector ground"
- note added: "PD_GND\n"
- moved on the sheet: C11, C12, C13, C14, C16, L2, R31, U8

Commit message: Updated PCB and generated gerbers
Parts:
- C11, C13: value 0.1µF -> 0.1u
- C12, C16: value 4.7µF -> 4.7u
- C14: value 5600pF -> 5600p
- C15: value 10µF 10V -> 10u
- C26: value 1µf 10V -> 1u
- L2: value 4.7µH -> 4.7u
Changed lines of the file:
@@
 P 3200 1400
 F 0 "C13" H 3315 1446 50  0000 L CNN
-F 1 "0.1µF" H 3315 1355 50  0000 L CNN
+F 1 "0.1u" H 3315 1355 50  0000 L CNN
 F 2 "Capacitor_SMD:C_0402_1005Metric" H 3238 1250 50  0001 C CNN
 F 3 "~" H 3200 1400 50  0001 C CNN
@@
 P 2600 1400
 F 0 "C11" H 2485 1446 50  0000 R CNN
-F 1 "0.1µF" H 2485 1355 50  0000 R CNN
+F 1 "0.1u" H 2485 1355 50  0000 R CNN
 F 2 "Capacitor_SMD:C_0402_1005Metric" H 2638 1250 50  0001 C CNN
 F 3 "~" H 2600 1400 50  0001 C CNN
@@
 P 1350 5150
 F 0 "C12" V 1098 5150 50  0000 C CNN
-F 1 "4.7µF" V 1189 5150 50  0000 C CNN
+F 1 "4.7u" V 1189 5150 50  0000 C CNN
 F 2 "Capacitor_SMD:C_0402_1005Metric" H 1388 5000 50  0001 C CNN
 F 3 "~" H 1350 5150 50  0001 C CNN
@@
 P 3500 5500
 F 0 "C14" V 3248 5500 50  0000 C CNN
-F 1 "5600pF" V 3339 5500 50  0000 C CNN
+F 1 "5600p" V 3339 5500 50  0000 C CNN
 F 2 "Capacitor_SMD:C_0402_1005Metric" H 3538 5350 50  0001 C CNN
 F 3 "~" H 3500 5500 50  0001 C CNN
@@
 P 3850 6200
 F 0 "L2" H 3850 6415 50  0000 C CNN
-F 1 "4.7µH" H 3850 6324 50  0000 C CNN
+F 1 "4.7u" H 3850 6324 50  0000 C CNN
 F 2 "Inductor_SMD:L_0603_1608Metric" H 3850 6200 50  0001 C CNN
 F 3 "~" H 3850 6200 50  0001 C CNN
@@
 P 4550 6200
 F 0 "C16" V 4298 6200 50  0000 C CNN
-F 1 "4.7µF" V 4389 6200 50  0000 C CNN
+F 1 "4.7u" V 4389 6200 50  0000 C CNN
 F 2 "Capacitor_SMD:C_0402_1005Metric" H 4588 6050 50  0001 C CNN
 F 3 "~" H 4550 6200 50  0001 C CNN
@@
 P 5250 2700
 F 0 "C15" V 5100 2700 50  0000 C CNN
-F 1 "10µF 10V" V 5400 2700 50  0000 C CNN
+F 1 "10u" V 5400 2700 50  0000 C CNN
 F 2 "Capacitor_SMD:C_0402_1005Metric" H 5288 2550 50  0001 C CNN
 F 3 "~" H 5250 2700 50  0001 C CNN
@@
 P 8650 2750
 F 0 "C26" H 8765 2796 50  0000 L CNN
-F 1 "1µf 10V" H 8765 2705 50  0000 L CNN
+F 1 "1u" H 8765 2705 50  0000 L CNN
 F 2 "Capacitor_SMD:C_0402_1005Metric" H 8688 2600 50  0001 C CNN
 F 3 "~" H 8650 2750 50  0001 C CNN
