File: CAD/IMUSensor.sch (KiCad schematic (older format))
At the start: 6 parts

Commit message: Finished PCB Draft -- waiting for review
Parts:
- removed C3: 100nF, symbol Device:C
- removed U?: LSM6DS33TR, PQFN50P300X300X86-16N, symbol LSM6DS33TR:LSM6DS33TR
- added U6: LSM6DS33TR, LSM6DS33TR:PQFN50P300X300X86-16N, symbol LSM6DS33TR:LSM6DS33TR
- C10: renamed from C4; footprint (none) -> Capacitor_SMD:C_0402_1005Metric
- C9: renamed from C2; footprint (none) -> Capacitor_SMD:C_0402_1005Metric
- Rpu1, Rpu2: renamed from Rpu; footprint (none) -> Resistor_SMD:R_0402_1005Metric
Connections:
- net CS: now also U6.5 (CS)
- net GND: now also U6.10 (RES), U6.11 (RES), U6.12 (GND), U6.13 (GND), U6.8 (RES), U6.9 (RES)
- net INT1: now also U6.7 (INT1)
- net INT2: now also U6.6 (INT2)
- net SCL: now also U6.2 (SCL)
- net SDA-SDISDO: now also U6.3 (SDA)
- net SDO-SA0: now also U6.4 (SDO/SA0)
- net VDD: now also U6.1 (VDDIO), U6.15 (RES), U6.16 (VDD)
Changed lines of the file:
@@
 EESchema Schematic File Version 4
-EELAYER 29 0
+LIBS:HealthMonitor-cache
+LIBS:Max86141-cache
+EELAYER 26 0
 EELAYER END
 $Descr A4 11693 8268
 encoding utf-8
-Sheet 1 1
+Sheet 4 7
 Title ""
 Date ""
@@
 	6950 3250 7350 3250
 $Comp
-L Device:C C2
+L Device:C C9
 U 1 1 5CD13038
 P 7350 3500
-F 0 "C2" H 7150 3500 50  0000 L CNN
+F 0 "C9" H 7150 3500 50  0000 L CNN
 F 1 "100nF" H 7100 3400 50  0000 L CNN
-F 2 "" H 7388 3350 50  0001 C CNN
+F 2 "Capacitor_SMD:C_0402_1005Metric" H 7388 3350 50  0001 C CNN
 F 3 "~" H 7350 3500 50  0001 C CNN
 	1    7350 3500
@@
 	6800 4150 6800 3900
 $Comp
-L power:VDD #PWR?
+L power:VDD #PWR035
 U 1 1 5CD16738
 P 7750 3700
-F 0 "#PWR?" H 7750 3550 50  0001 C CNN
+F 0 "#PWR035" H 7750 3550 50  0001 C CNN
 F 1 "VDD" H 7767 3873 50  0000 C CNN
 F 2 "" H 7750 3700 50  0001 C CNN
@@
 $EndComp
 $Comp
-L Device:C C4
+L Device:C C10
 U 1 1 5CD1707B
 P 7750 4100
-F 0 "C4" H 7865 4146 50  0000 L CNN
+F 0 "C10" H 7865 4146 50  0000 L CNN
 F 1 "10µF" H 7865 4055 50  0000 L CNN
-F 2 "" H 7788 3950 50  0001 C CNN
+F 2 "Capacitor_SMD:C_0402_1005Metric" H 7788 3950 50  0001 C CNN
 F 3 "~" H 7750 4100 50  0001 C CNN
 	1    7750 4100
@@
 	6800 3900 7750 3900
 $Comp
-L Device:C C3
-U 1 1 5CD1854A
-P 7200 4100
-F 0 "C3" H 7315 4146 50  0000 L CNN
-F 1 "100nF" H 7315 4055 50  0000 L CNN
-F 2 "" H 7238 3950 50  0001 C CNN
-F 3 "~" H 7200 4100 50  0001 C CNN
-	1    7200 4100
-	1    0    0    -1
-$EndComp
-Wire Wire Line
-	7200 3950 7750 3950
-$Comp
-L power:GND #PWR?
+L power:GND #PWR036
 U 1 1 5CD19977
 P 7750 4250
-F 0 "#PWR?" H 7750 4000 50  0001 C CNN
+F 0 "#PWR036" H 7750 4000 50  0001 C CNN
 F 1 "GND" H 7755 4077 50  0000 C CNN
 F 2 "" H 7750 4250 50  0001 C CNN
@@
 	1    0    0    -1
 $EndComp
-$Comp
-L power:GND #PWR?
-U 1 1 5CD19E78
-P 7200 4250
-F 0 "#PWR?" H 7200 4000 50  0001 C CNN
-F 1 "GND" H 7205 4077 50  0000 C CNN
-F 2 "" H 7200 4250 50  0001 C CNN
-F 3 "" H 7200 4250 50  0001 C CNN
-	1    7200 4250
-	1    0    0    -1
-$EndComp
 Wire Wire Line
 	6550 4300 6800 4300
@@
 	6450 5100 6450 5250
 $Comp
-L power:GND #PWR?
+L power:GND #PWR031
 U 1 1 5CD1DDAF
 P 6450 5250
-F 0 "#PWR?" H 6450 5000 50  0001 C CNN
+F 0 "#PWR031" H 6450 5000 50  0001 C CNN
 F 1 "GND" H 6455 5077 50  0000 C CNN
 F 2 "" H 6450 5250 50  0001 C CNN
@@
 	7350 3100 7350 3250
 $Comp
-L power:VDD #PWR?
+L power:VDD #PWR033
 U 1 1 5CD13849
 P 7350 3100
-F 0 "#PWR?" H 7350 2950 50  0001 C CNN
+F 0 "#PWR033" H 7350 2950 50  0001 C CNN
 F 1 "VDD" H 7367 3273 50  0000 C CNN
 F 2 "" H 7350 3100 50  0001 C CNN
@@
 	5200 4150 5350 4150
 $Comp
-L power:GND #PWR?
+L power:GND #PWR034
 U 1 1 5CD1403B
 P 7350 3650
-F 0 "#PWR?" H 7350 3400 50  0001 C CNN
+F 0 "#PWR034" H 7350 3400 50  0001 C CNN
 F 1 "GND" H 7355 3477 50  0000 C CNN
 F 2 "" H 7350 3650 50  0001 C CNN
@@
 	1    0    0    -1
 $EndComp
-$Comp
-L LSM6DS33TR:LSM6DS33TR U?
-U 1 1 5CD0DE35
+Wire Wire Line
+	7750 3950 7750 3900
+Wire Wire Line
+	7750 3900 7750 3700
+Connection ~ 7750 3900
+Connection ~ 7750 3700
+Wire Wire Line
+	7350 3100 7550 3100
+Wire Wire Line
+	7550 3100 7550 3700
+Wire Wire Line
+	6150 3550 6150 3600
+Wire Wire Line
+	6200 3450 6050 3450
+Wire Wire Line
+	6050 3000 6050 3450
+Connection ~ 6050 3450
+Wire Wire Line
+	6050 3450 6050 3600
+Wire Wire Line
+	6150 3550 6950 3550
+$Comp
+L Device:R Rpu1
+U 1 1 5CD31892
+P 6350 3450
+F 0 "Rpu1" V 6350 3450 50  0000 C CNN
+F 1 "10kOhms" V 6250 3450 50  0000 C CNN
+F 2 "Resistor_SMD:R_0402_1005Metric" V 6280 3450 50  0001 C CNN
+F 3 "~" H 6350 3450 50  0001 C CNN
+	1    6350 3450
+	0    1    1    0
+$EndComp
+Wire Wire Line
+	6500 3450 6950 3450
+Connection ~ 6950 3450
+Wire Wire Line
+	6950 3450 6950 3250
+$Comp
+L Device:R Rpu2
+U 1 1 5CD349A4
+P 6500 3250
+F 0 "Rpu2" V 6500 3250 50  0000 C CNN
+F 1 "10kOhms" V 6400 3250 50  0000 C CNN
+F 2 "Resistor_SMD:R_0402_1005Metric" V 6430 3250 50  0001 C CNN
+F 3 "~" H 6500 3250 50  0001 C CNN
+	1    6500 3250
+	0    1    1    0
+$EndComp
+Wire Wire Line
+	5950 3250 6350 3250
+Wire Wire Line
+	6650 3250 6950 3250
+Connection ~ 6950 3250
+Connection ~ 5950 3250
+Wire Wire Line
+	5950 3250 5950 3600
+Wire Wire Line
+	5950 3000 5950 3250
+$Comp
+L LSM6DS33TR:LSM6DS33TR U6
+U 1 1 5CD83675
 P 5950 4300
-F 0 "U?" H 5900 4300 50  0000 L CNN
-F 1 "LSM6DS33TR" H 5750 4200 43  0000 L CIN
-F 2 "PQFN50P300X300X86-16N" H 5350 3100 50  0001 L BNN
-F 3 "" H 6750 3550 50  0001 L BNN
+F 0 "U6" H 5900 4350 50  0000 L CNN
+F 1 "LSM6DS33TR" H 5750 4250 43  0000 L CIN
+F 2 "LSM6DS33TR:PQFN50P300X300X86-16N" H 5350 3100 50  0001 L BNN
+F 3 "STMicroelectronics" H 6750 3550 50  0001 L BNN
 F 4 "Integrated Circuit, Misc s 3d Accelerometer And Gyro Lsm6ds3" H 5350 3100 50  0001 L BNN "Field5"
 F 5 "LSM6DS33TR" H 6750 3550 50  0001 L BNN "Field6"
@@
 	1    0    0    -1
 $EndComp
-Wire Wire Line
-	7750 3950 7750 3900
-Connection ~ 7750 3950
-Wire Wire Line
-	7750 3900 7750 3700
-Connection ~ 7750 3900
-Connection ~ 7750 3700
-Wire Wire Line
-	7350 3100 7550 3100
-Wire Wire Line
-	7550 3100 7550 3700
-Wire Wire Line
-	6150 3550 6150 3600
-Wire Wire Line
-	6200 3450 6050 3450
-Wire Wire Line
-	6050 3000 6050 3450
-Connection ~ 6050 3450
-Wire Wire Line
-	6050 3450 6050 3600
-Wire Wire Line
-	6150 3550 6950 3550
-$Comp
-L Device:R Rpu
-U 1 1 5CD31892
-P 6350 3450
-F 0 "Rpu" V 6350 3450 50  0000 C CNN
-F 1 "10kOhms" V 6250 3450 50  0000 C CNN
-F 2 "" V 6280 3450 50  0001 C CNN
-F 3 "~" H 6350 3450 50  0001 C CNN
-	1    6350 3450
-	0    1    1    0
-$EndComp
-Wire Wire Line
-	6500 3450 6950 3450
-Connection ~ 6950 3450
-Wire Wire Line
-	6950 3450 6950 3250
-$Comp
-L Device:R Rpu
-U 1 1 5CD349A4
-P 6500 3250
-F 0 "Rpu" V 6500 3250 50  0000 C CNN
-F 1 "10kOhms" V 6400 3250 50  0000 C CNN
-F 2 "" V 6430 3250 50  0001 C CNN
-F 3 "~" H 6500 3250 50  0001 C CNN
-	1    6500 3250
-	0    1    1    0
-$EndComp
-Wire Wire Line
-	5950 3250 6350 3250
-Wire Wire Line
-	6650 3250 6950 3250
-Connection ~ 6950 3250
-Connection ~ 5950 3250
-Wire Wire Line
-	5950 3250 5950 3600
-Wire Wire Line
-	5950 3000 5950 3250
+Text HLabel 6600 5100 2    50   UnSpc ~ 0
+GND
+Wire Wire Line
+	6600 5100 6450 5100
+Connection ~ 6450 5100
 $EndSCHEMATC

Commit message: rescue commit
Parts:
- removed U6: LSM6DS33TR, LSM6DS33TR:PQFN50P300X300X86-16N, symbol LSM6DS33TR:LSM6DS33TR
- added U6: LSM6DSLTR, LSM6DSLTR:PQFN50P300X250X86-14N, symbol LSM6DSLTR:LSM6DSLTR
- C10: value 10µF -> 100nF
Connections:
- net GND: now also U6.1 (SDO/SA0), U6.6 (GND), U6.7 (GND)
- net INT1: now also U6.4 (INT1)
- net INT2: now also U6.9 (INT2)
- net SCL: now also Rpu1.1, U6.13 (SCL); no longer Rpu1.2
- net VDD: now also Rpu1.2, U6.12 (CS), U6.5 (VDDIO), U6.8 (VDD); no longer Rpu1.1
- net SDA-SDISDO renamed SDA
- net SDA: now also U6.14 (SDA)
- no-connect marks 0 -> 2
