File: CAD/SoC.sch (KiCad schematic (older format))
At the start: 11 parts, among them J7 Conn_02x05_Odd_Even, U10 AT24CS02-XHM, U11 BT832L, Y1 ABS06-32.768KHZ-T

Commit message: rescue commit
Parts:
- added C29, C30: 12p, Capacitor_SMD:C_0402_1005Metric, symbol Device:C
- added J27: MOLEX_51281-0594MOLEX_51281-0594_0_0, Molex - 51281-0594:Molex - 51281-0594-MOLEX_51281-0594_0, symbol Molex~-~51281-0594:MOLEX_51281-0594MOLEX_51281-0594_0_0
- added J28, J29: Conn_01x01_Male, Connector_PinHeader_1.27mm:PinHeader_1x01_P1.27mm_Vertical, symbol Connector:Conn_01x01_Male
Connections:
- wire segments 97 -> 117
Changed lines of the file:
@@
 Wire Wire Line
 	5550 5100 5550 4750
+Wire Wire Line
+	4600 3900 4400 3900
+$Comp
+L Connector:Conn_01x01_Male J28
+U 1 1 5CEF8F8A
+P 3500 4100
+F 0 "J28" H 3606 4278 50  0000 C CNN
+F 1 "Conn_01x01_Male" H 3606 4187 50  0000 C CNN
+F 2 "Connector_PinHeader_1.27mm:PinHeader_1x01_P1.27mm_Vertical" H 3500 4100 50  0001 C CNN
+F 3 "~" H 3500 4100 50  0001 C CNN
+	1    3500 4100
+	1    0    0    -1
+$EndComp
+$Comp
+L Connector:Conn_01x01_Male J29
+U 1 1 5CEF8FEE
+P 3500 4300
+F 0 "J29" H 3606 4478 50  0000 C CNN
+F 1 "Conn_01x01_Male" H 3606 4387 50  0000 C CNN
+F 2 "Connector_PinHeader_1.27mm:PinHeader_1x01_P1.27mm_Vertical" H 3500 4300 50  0001 C CNN
+F 3 "~" H 3500 4300 50  0001 C CNN
+	1    3500 4300
+	1    0    0    -1
+$EndComp
+Wire Wire Line
+	3700 4100 4250 4100
+Wire Wire Line
+	4250 4100 4250 3750
+Connection ~ 4250 3750
+Wire Wire Line
+	4250 3750 4600 3750
+Wire Wire Line
+	3700 4300 4400 4300
+Wire Wire Line
+	4400 4300 4400 3900
+$Comp
+L Molex~-~51281-0594:MOLEX_51281-0594MOLEX_51281-0594_0_0 J27
+U 1 1 5CF01441
+P 1850 4100
+F 0 "J27" V 2820 3691 45  0000 C CNN
+F 1 "MOLEX_51281-0594MOLEX_51281-0594_0_0" H 1850 4100 45  0001 L BNN
+F 2 "Molex - 51281-0594:Molex - 51281-0594-MOLEX_51281-0594_0" H 1880 4250 20  0001 C CNN
+F 3 "" H 1850 4100 50  0001 C CNN
+	1    1850 4100
+	0    -1   -1   0
+$EndComp
+Wire Wire Line
+	2600 3750 3150 3750
+Wire Wire Line
+	2600 3900 2450 3900
+Wire Wire Line
+	2600 3750 2600 3900
+Wire Wire Line
+	4400 3700 4400 3900
+Wire Wire Line
+	2450 3700 2750 3700
+Connection ~ 4400 3900
+$Comp
+L Device:C C29
+U 1 1 5CF11FCD
+P 2750 4000
+F 0 "C29" V 2498 4000 50  0000 C CNN
+F 1 "12p" V 2589 4000 50  0000 C CNN
+F 2 "Capacitor_SMD:C_0402_1005Metric" H 2788 3850 50  0001 C CNN
+F 3 "~" H 2750 4000 50  0001 C CNN
+	1    2750 4000
+	-1   0    0    1
+$EndComp
+$Comp
+L Device:C C30
+U 1 1 5CF1203E
+P 3150 4000
+F 0 "C30" V 2898 4000 50  0000 C CNN
+F 1 "12p" V 2989 4000 50  0000 C CNN
+F 2 "Capacitor_SMD:C_0402_1005Metric" H 3188 3850 50  0001 C CNN
+F 3 "~" H 3150 4000 50  0001 C CNN
+	1    3150 4000
+	-1   0    0    1
+$EndComp
+Wire Wire Line
+	2750 3850 2750 3700
+Connection ~ 2750 3700
+Wire Wire Line
+	2750 3700 4400 3700
+Wire Wire Line
+	3150 3850 3150 3750
+Connection ~ 3150 3750
+Wire Wire Line
+	3150 3750 4250 3750
+$Comp
+L power:GND #PWR0130
+U 1 1 5CF17D92
+P 2950 4250
+F 0 "#PWR0130" H 2950 4000 50  0001 C CNN
+F 1 "GND" H 2955 4077 50  0000 C CNN
+F 2 "" H 2950 4250 50  0001 C CNN
+F 3 "" H 2950 4250 50  0001 C CNN
+	1    2950 4250
+	1    0    0    -1
+$EndComp
+Wire Wire Line
+	2950 4250 2950 4200
+Wire Wire Line
+	2950 4200 2750 4200
+Wire Wire Line
+	2750 4200 2750 4150
+Wire Wire Line
+	2950 4200 3150 4200
+Wire Wire Line
+	3150 4200 3150 4150
+Connection ~ 2950 4200
 $EndSCHEMATC
