File: CAD/power.sch (KiCad schematic (older format))
At the start: 28 parts, among them J1 USB_C_Receptacle_USB2.0, U1 ADP5092ACPZ-1-R7, U2 LTC4079IDD-PBF

Commit message: Finished PCB Draft -- waiting for review
Parts:
- added C1: 0.1u, Capacitor_SMD:C_0402_1005Metric, symbol Device:C
- added C24, C25: 1u, Capacitor_SMD:C_0402_1005Metric, symbol Device:C
- added R10, R11, R35: 10k, Resistor_SMD:R_0402_1005Metric, symbol Device:R
- added R6: 1M, Resistor_SMD:R_0402_1005Metric, symbol Device:R
- added R7: 2M, Resistor_SMD:R_0402_1005Metric, symbol Device:R
- added U1: MAX17048G+T10, footprints:MAX17048G+, symbol MAX17048G+:MAX17048G+T10
- added U13: ADG884BRMZ, footprints:ADG884BRMZ, symbol ADG884BRMZ:ADG884BRMZ
- added U4: LD39015M33R, Package_TO_SOT_SMD:SOT-23-5, symbol Regulator_Linear:LD39015M33R
- R19: renamed from R15; value 3.57M -> 3.32M
- R21: renamed from R17; value 6.49M -> 6.65M
- renumbered C1 to C2, C2 to C3, C3 to C4, C4 to C5, C5 to C6, J1 to J6, R8 to R12, R9 to R13, R10 to R14, R11 to R15, R12 to R16, R13 to R17, R14 to R18, R16 to R20, R18 to R22, R6 to R8, R7 to R9, U1 to U2, U2 to U3
Connections:
- net +3V3: now also R10.1, R11.1, U13.3 (D1); no longer C3.1, U2.14 (REG_OUT), U2.15 (REF_FB)
- net BAT+: now also C1.2, R35.2, U1.2 (CELL), U1.3 (VDD), U13.9 (D2); no longer R18.2, U2.17 (BAT), U3.10 (BAT)
- net GND: now also C1.1, C24.2, C25.2, R7.2, U1.1 (CTG), U1.4 (GND), U1.6 (QSTRT), U1.9 (EPAD), U13.6 (GND), U4.2 (GND)
- net USB_VBUS: now reaches C5.1, J6.A4 (VBUS), J6.A9 (VBUS), J6.B4 (VBUS), J6.B9 (VBUS), U3.1 (IN), U3.2 (EN)
- net USB_VBUS: now also C24.1, R6.1, U4.1 (IN), U4.3 (EN)
- net USBD+: now reaches J6.A6 (D+)
- net USBD-: now reaches J6.A7 (D-)
- new net: R35.1, U13.1 (VDD)
- new net BAT_EH: U13.7 (S2B), U2.17 (BAT)
- new net BAT_USB: R18.2, U13.10 (S2A), U3.10 (BAT)
- new net B_CONN: R6.2, R7.1, U13.4 (IN1), U13.8 (IN2)
- new net EH_3v3: C3.1, U13.5 (S1B), U2.14 (REG_OUT), U2.15 (REF_FB)
- new net SCL_BAT_STATUS: R10.2, U1.7 (SCL)
- new net SDA_BAT_STATUS: R11.2, U1.8 (SDA)
- new net USB_3v3: C25.1, U13.2 (S1A), U4.5 (OUT)
- no-connect marks 1 -> 7
Other:
- moved on the sheet: C2, C3, C4, C5, C6, FB1, J6, L1, R1, R12, R13, R14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

Commit message: Generated gerbers
Parts:
- J6: footprint Connector_USB:USB_C_Receptacle_Amphenol_12401610E4-2A_CircularHoles -> footprints:USB_C_Receptacle_Amphenol_12401610E4-2A_CircularHoles
Changed lines of the file:
@@
 EESchema Schematic File Version 4
 LIBS:HealthMonitor-cache
-LIBS:Max86141-cache
 EELAYER 26 0
 EELAYER END
@@
 F 0 "J6" H 2755 5117 50  0000 C CNN
 F 1 "USB_C_Receptacle_USB2.0" H 2755 5026 50  0000 C CNN
-F 2 "Connector_USB:USB_C_Receptacle_Amphenol_12401610E4-2A_CircularHoles" H 2800 4250 50  0001 C CNN
+F 2 "footprints:USB_C_Receptacle_Amphenol_12401610E4-2A_CircularHoles" H 2800 4250 50  0001 C CNN
 F 3 "https://www.usb.org/sites/default/files/documents/usb_type-c.zip" H 2800 4250 50  0001 C CNN
 	1    2650 4250

Commit message: rescue commit
Parts:
- added C28, C8: 1u, Capacitor_SMD:C_0402_1005Metric, symbol Device:C
- added J26: Conn_01x01_Male, Connector_PinHeader_1.27mm:PinHeader_1x01_P1.27mm_Vertical, symbol Connector:Conn_01x01_Male
- added R37: 0, Resistor_SMD:R_0402_1005Metric, symbol Device:R
- added U14: LD39015M33R, Package_TO_SOT_SMD:SOT-23-5, symbol Regulator_Linear:LD39015M33R
Connections:
- net BAT+: now also R37.2
- net GND: now also C28.2, C8.2, U14.2 (GND)
- new net: C8.1, R37.1, U14.1 (IN), U14.3 (EN)
- new net: C28.1, J26.1 (Pin_1), U14.5 (OUT)
Changed lines of the file:
@@
 L power:+3V3 #PWR05
 U 1 1 5CD686A5
-P 8350 2850
-F 0 "#PWR05" H 8350 2700 50  0001 C CNN
-F 1 "+3V3" V 8400 2900 50  0000 L CNN
-F 2 "" H 8350 2850 50  0001 C CNN
-F 3 "" H 8350 2850 50  0001 C CNN
-	1    8350 2850
+P 8050 2850
+F 0 "#PWR05" H 8050 2700 50  0001 C CNN
+F 1 "+3V3" V 8100 2900 50  0000 L CNN
+F 2 "" H 8050 2850 50  0001 C CNN
+F 3 "" H 8050 2850 50  0001 C CNN
+	1    8050 2850
 	0    -1   -1   0
 $EndComp
@@
 BAT_EH
 Wire Wire Line
-	7900 3950 7900 3600
-Wire Wire Line
 	7900 3600 8200 3600
 Connection ~ 7900 3950
@@
 Wire Wire Line
 	10850 3150 10750 3150
-Wire Wire Line
-	8350 2850 8550 2850
 Text Label 2850 950  2    50   ~ 0
 EH_3v3
@@
 Wire Wire Line
 	3950 5500 3950 5400
+$Comp
+L Regulator_Linear:LD39015M33R U14
+U 1 1 5CEEC16E
+P 9850 5100
+F 0 "U14" H 9850 5442 50  0000 C CNN
+F 1 "LD39015M33R" H 9850 5351 50  0000 C CNN
+F 2 "Package_TO_SOT_SMD:SOT-23-5" H 9850 5425 50  0001 C CIN
+F 3 "http://www.st.com/resource/en/datasheet/ld39015.pdf" H 9850 5100 50  0001 C CNN
+	1    9850 5100
+	1    0    0    -1
+$EndComp
+Wire Wire Line
+	9550 5100 9400 5100
+Wire Wire Line
+	9400 5100 9400 5000
+Wire Wire Line
+	9400 5000 9550 5000
+Wire Wire Line
+	9400 5000 9300 5000
+Connection ~ 9400 5000
+$Comp
+L power:GND #PWR0127
+U 1 1 5CEEC17B
+P 9850 5450
+F 0 "#PWR0127" H 9850 5200 50  0001 C CNN
+F 1 "GND" H 9855 5277 50  0000 C CNN
+F 2 "" H 9850 5450 50  0001 C CNN
+F 3 "" H 9850 5450 50  0001 C CNN
+	1    9850 5450
+	1    0    0    -1
+$EndComp
+Wire Wire Line
+	9850 5450 9850 5400
+$Comp
+L Device:C C8
+U 1 1 5CEEC184
+P 9300 5200
+F 0 "C8" H 9100 5250 50  0000 L CNN
+F 1 "1u" H 9100 5150 50  0000 L CNN
+F 2 "Capacitor_SMD:C_0402_1005Metric" H 9338 5050 50  0001 C CNN
+F 3 "~" H 9300 5200 50  0001 C CNN
+	1    9300 5200
+	1    0    0    -1
+$EndComp
+$Comp
+L Device:C C28
+U 1 1 5CEEC18B
+P 10200 5200
+F 0 "C28" H 10300 5250 50  0000 L CNN
+F 1 "1u" H 10300 5150 50  0000 L CNN
+F 2 "Capacitor_SMD:C_0402_1005Metric" H 10238 5050 50  0001 C CNN
+F 3 "~" H 10200 5200 50  0001 C CNN
+	1    10200 5200
+	1    0    0    -1
+$EndComp
+Wire Wire Line
+	10200 5050 10200 5000
+Wire Wire Line
+	9300 5050 9300 5000
+Connection ~ 9300 5000
+$Comp
+L power:GND #PWR0128
+U 1 1 5CEEC198
+P 9300 5450
+F 0 "#PWR0128" H 9300 5200 50  0001 C CNN
+F 1 "GND" H 9305 5277 50  0000 C CNN
+F 2 "" H 9300 5450 50  0001 C CNN
+F 3 "" H 9300 5450 50  0001 C CNN
+	1    9300 5450
+	1    0    0    -1
+$EndComp
+$Comp
+L power:GND #PWR0129
+U 1 1 5CEEC19E
+P 10200 5450
+F 0 "#PWR0129" H 10200 5200 50  0001 C CNN
+F 1 "GND" H 10205 5277 50  0000 C CNN
+F 2 "" H 10200 5450 50  0001 C CNN
+F 3 "" H 10200 5450 50  0001 C CNN
+	1    10200 5450
+	1    0    0    -1
+$EndComp
+Wire Wire Line
+	10200 5450 10200 5350
+Wire Wire Line
+	9300 5450 9300 5350
+$Comp
+L Device:R R37
+U 1 1 5CEF6603
+P 8750 5000
+F 0 "R37" V 8800 4850 50  0000 C CNN
+F 1 "0" V 8800 5200 50  0000 C CNN
+F 2 "Resistor_SMD:R_0402_1005Metric" V 8680 5000 50  0001 C CNN
+F 3 "~" H 8750 5000 50  0001 C CNN
+	1    8750 5000
+	0    1    1    0
+$EndComp
+Wire Wire Line
+	7900 3600 7900 3950
+Text Label 8450 4950 2    50   ~ 0
+BAT
+Wire Wire Line
+	8450 4950 8450 5000
+Wire Wire Line
+	8450 5000 8600 5000
+Wire Wire Line
+	8900 5000 9300 5000
+$Comp
+L Connector:Conn_01x01_Male J26
+U 1 1 5CF7F686
+P 10700 5000
+F 0 "J26" H 10806 5178 50  0000 C CNN
+F 1 "Conn_01x01_Male" V 10806 5087 50  0000 C CNN
+F 2 "Connector_PinHeader_1.27mm:PinHeader_1x01_P1.27mm_Vertical" H 10700 5000 50  0001 C CNN
+F 3 "~" H 10700 5000 50  0001 C CNN
+	1    10700 5000
+	-1   0    0    1
+$EndComp
+Wire Wire Line
+	10200 5000 10500 5000
+Wire Wire Line
+	10150 5000 10200 5000
+Connection ~ 10200 5000
+Wire Wire Line
+	8050 2850 8550 2850
 $EndSCHEMATC
